File: Power_Supply_Schematic.kicad_sch (KiCad schematic)
At the start: 11 parts, among them J1 Conn_01x02, J2 Barrel_Jack_Switch_Pin3Ring, U3 AMS1117-3.3, U4 AMS1117-3.3

Commit message: Changes done as per Poineer Circuits
Parts:
- added D20, D21: LED, LED_SMD:LED_0805_2012Metric_Pad1.15x1.40mm_HandSolder, symbol Device:LED
- added R47, R48: 4.7K, Resistor_SMD:R_0805_2012Metric_Pad1.20x1.40mm_HandSolder, symbol Device:R_US
Connections:
- net +3.3V: now also R47.2
- net +ADE_3.3V: now also R48.2
- net ADE_GND: now also D21.1 (K)
- net GND: now also D20.1 (K)
- new net: D21.2 (A), R48.1
- new net: D20.2 (A), R47.1
