File: STM32_Schematic.kicad_sch (KiCad schematic)
At the start: 44 parts, among them J12 Conn_01x06_Pin, J13 Conn_01x08_Pin, J14 Conn_01x08_Pin, J15 Conn_01x08_Pin, J16 Conn_01x08_Pin, J17 Conn_01x08_Pin, J18 Conn_01x08_Pin, J19 Conn_01x03_Pin, J20 Conn_01x03_Pin, J21 Conn_01x03_Pin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

Commit message: Changes done as per Poineer Circuits
Parts:
- added J11: Conn_01x02, Connector_PinSocket_2.54mm:PinSocket_1x02_P2.54mm_Vertical, symbol Connector_Generic:Conn_01x02
Connections:
- net +3.3V: now also J11.1 (Pin_1)
- net GND: now also J11.2 (Pin_2)
